Commit message: joint_state updates

File: src/alfie_urdf/urdf/alfiebot.urdf (robot description, URDF)
Before this commit: robot alfiebot.021.urdf, 23 links, 22 joints
Links:
- link neck3_link: geometry visual mesh filename=file:///home/alansrobotlab/Downloads/urdf/urdf/meshes/activ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 scale=1. 1. 1.; visual mesh filename=file:///home/alansrobotlab/Downloads/urdf/urdf/meshes/neck3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 scale=1. 1. 1.
Joints:
- joint head_pitch_joint: axis 0. 0. 1. -> 0. 0. -1.; origin xyz=-0.01875 -0. 0.053  rpy=1.5707964 0. 1.5707964 -> xyz=-0.01875 -0. 0.053  rpy=1.5707964 0.0 1.5707964
- joint head_yaw_joint: origin xyz=-0.0011403 0.0054173 0.8706568 rpy=0. 0. -0.0025961 -> xyz=-0.0011403 0.0054173 0.8706568 rpy=0.0 0.0 0.0
- joint left_elbow_pitch_joint: origin xyz=0.2368151 -0.0300024 0.0193  rpy=0.0000002 0. 1.5707964 -> xyz=0.2368151 -0.0300024 0.0193  rpy=0. 0. 1.5707964

Commit message: urdf rendered correctly; laggy; no tf

File: src/alfie_urdf/urdf/alfiebot.urdf (robot description, URDF)
Before this commit: robot alfiebot.021.urdf, 23 links, 22 joints
Links:
- link back_link: geometry visual mesh filename=package://alfie_urdf/meshes/back_frame.obj scale=1. 1. 1.; visual mesh filename=package://alfie_urdf/meshes/left_shoulder.obj scale=1. 1. 1.
- link base_link: geometry visual mesh filename=package://alfie_urdf/meshes/6010_battery.obj scale=1. 1. 1.; visual mesh filename=package://alfie_urdf/meshes/back_servo_cover.obj scale=1. 1. 1.
- link head_link: geometry visual mesh filename=package://alfie_urdf/meshes/active_horn.obj scale=1. 1. 1.; visual mesh filename=package://alfie_urdf/meshes/eye_frame.obj scale=1. 1. 1.
- link left_arm_lower_link: geometry visual mesh filename=package://alfie_urdf/meshes/active_horn.obj scale=1. 1. 1.; visual mesh filename=package://alfie_urdf/meshes/active_horn.obj scale=1. 1. 1.
- link left_arm_upper_link: geometry visual mesh filename=package://alfie_urdf/meshes/upper_frame.obj scale=1. 1. 1.
- link left_gripper_active_link: geometry collision mesh filename=package://alfie_urdf/meshes/gripper_active_collision.obj scale=1. 1. 1.; visual mesh filename=package://alfie_urdf/meshes/gripper.obj scale=1. 1. 1.
- link left_gripper_passive_link: geometry collision mesh filename=package://alfie_urdf/meshes/gripper_passive_collision.obj scale=1. 1. 1.; visual mesh filename=package://alfie_urdf/meshes/gripper.obj scale=1. 1. 1.
- link left_hand_link: geometry visual mesh filename=package://alfie_urdf/meshes/hand_frame.obj scale=1. 1. 1.; visual mesh filename=package://alfie_urdf/meshes/st3215.obj scale=1. 1. 1.
- link left_shoulder_link: geometry visual mesh filename=package://alfie_urdf/meshes/active_horn.obj scale=1. 1. 1.; visual mesh filename=package://alfie_urdf/meshes/active_horn.obj scale=1. 1. 1.
- link left_wrist_link: geometry visual mesh filename=package://alfie_urdf/meshes/active_horn.obj scale=1. 1. 1.; visual mesh filename=package://alfie_urdf/meshes/st3215.obj scale=1. 1. 1.
- link mecanum_fl_link: geometry collision mesh filename=package://alfie_urdf/meshes/roller.obj scale=1. 1. 1.; collision mesh filename=package://alfie_urdf/meshes/roller.obj scale=1. 1. 1.
- link mecanum_fr_link: geometry collision mesh filename=package://alfie_urdf/meshes/roller.obj scale=1. 1. 1.; collision mesh filename=package://alfie_urdf/meshes/roller.obj scale=1. 1. 1.
- link mecanum_rl_link: geometry collision mesh filename=package://alfie_urdf/meshes/roller.obj scale=1. 1. 1.; collision mesh filename=package://alfie_urdf/meshes/roller.obj scale=1. 1. 1.
- link mecanum_rr_link: geometry collision mesh filename=package://alfie_urdf/meshes/roller.obj scale=1. 1. 1.; collision mesh filename=package://alfie_urdf/meshes/roller.obj scale=1. 1. 1.
- link neck2_link: geometry visual mesh filename=package://alfie_urdf/meshes/neck2_frame.obj scale=1. 1. 1.
- link neck3_link: geometry visual mesh filename=package://alfie_urdf/meshes/active_horn.obj scale=1. 1. 1.; visual mesh filename=package://alfie_urdf/meshes/neck3_frame.obj scale=1. 1. 1.
- link right_arm_lower_link: geometry visual mesh filename=package://alfie_urdf/meshes/active_horn.obj scale=1. 1. 1.; visual mesh filename=package://alfie_urdf/meshes/active_horn.obj scale=1. 1. 1.
- link right_arm_upper_link: geometry visual mesh filename=package://alfie_urdf/meshes/upper_frame.obj scale=1. 1. 1.
- link right_gripper_active_link: geometry collision mesh filename=package://alfie_urdf/meshes/gripper_active_collision.obj scale=1. 1. 1.; visual mesh filename=package://alfie_urdf/meshes/gripper.obj scale=1. 1. 1.
- link right_gripper_passive_link: geometry collision mesh filename=package://alfie_urdf/meshes/gripper_passive_collision.obj scale=1. 1. 1.; visual mesh filename=package://alfie_urdf/meshes/gripper.obj scale=1. 1. 1.
- link right_hand_link: geometry visual mesh filename=package://alfie_urdf/meshes/hand_frame.obj scale=1. 1. 1.; visual mesh filename=package://alfie_urdf/meshes/st3215.obj scale=1. 1. 1.
- link right_shoulder_link: geometry visual mesh filename=package://alfie_urdf/meshes/active_horn.obj scale=1. 1. 1.; visual mesh filename=package://alfie_urdf/meshes/active_horn.obj scale=1. 1. 1.
- link right_wrist_link: geometry visual mesh filename=package://alfie_urdf/meshes/active_horn.obj scale=1. 1. 1.; visual mesh filename=package://alfie_urdf/meshes/st3215.obj scale=1. 1. 1.

Commit message: urdf update, reference package, add some color

File: src/alfie_urdf/urdf/alfiebot.urdf (robot description, URDF)
Before this commit: robot alfiebot, 23 links, 22 joints
Links:
- link base_link: geometry visual mesh filename=package://alfie_urdf/meshes/6010_battery.obj scale=1. 1. 1.; visual mesh filename=package://alfie_urdf/meshes/back_servo_cover.obj scale=1. 1. 1.
