Commit message: urdf: back joint zero raised 50mm, range 0-0.35m
Co-Authored-By: Claude Opus 5.5 <noreply@anthropic.com>

File: src/alfie_urdf/urdf/alfiebot.urdf (robot description, URDF)
Before this commit: robot alfiebot, 23 links, 22 joints
Joints:
- joint back_joint: limit lower=0. upper=0.39 effort=10000000. velocity=0. -> lower=0. upper=0.35 effort=10000000. velocity=0.; origin xyz=-0.001102 0.0016674 0.3291568 rpy=0. 0. 3.1415927 -> xyz=-0.001102 0.0016674 0.3791568 rpy=0. 0. 3.1415927
